File: ECAD/Designs/PCB001-0A_processorBoard/main_processor.kicad_sch (KiCad schematic)
At the start: 25 parts, among them J1 USB_C_Receptacle_USB2.0_16P, SW1 BSL, SW2 RST, U1 W25Q128JVP, U2 RP2350B-QFN80, Y1 ABM8-272-T3

Commit message: added off board sensors page, included more gpio (see google drive), and tracked the gpio better
Connections:
- net GPIO25 renamed LED_BUILTIN
Changed lines of the file:
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@@
-		)
-	)
-	(label "GPIO25"
-		(at 58.42 149.86 90)
-		(effects
-			(font
-				(size 1.27 1.27)
-			)
-			(justify left bottom)
 		)
 	)
@@
 		)
 	)
+	(label "LED_BUILTIN"
+		(at 58.42 149.86 90)
+		(effects
+			(font
+				(size 1.27 1.27)
+			)
+			(justify left bottom)
+		)
+	)
