File: ECAD/Designs/PCB001_processorBoard/PCB001-0A_processorBoard/on_board_comms.kicad_sch (KiCad schematic)
At the start: 4 parts

Commit message: added more connectors to the side of the PCB, added a basic power supply, and began putting parts on the PCB.
Parts:
- gave numbers to parts that had none: 4
Changed lines of the file:
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@@
 		(dnp no)
 		(fields_autoplaced yes)
-		(property "Reference" "#PWR044"
+		(property "Reference" "#PWR040"
 			(at 50.8 127 0)
 			(effects
@@
 		)
 		(pin "1"
+		)
+		(instances
+			(project "PCB001-0A_processorBoard"
+				(path "/c85d256f-82d8-4180-ad51-faa565e237b8/421006c7-5c19-4fe4-b045-335315607d2c"
+					(reference "#PWR040")
+					(unit 1)
+				)
+			)
 		)
 	)
@@
 		(dnp no)
 		(fields_autoplaced yes)
-		(property "Reference" "J?"
+		(property "Reference" "J5"
 			(at 43.18 123.19 0)
 			(effects
@@
 			(project "PCB001-0A_processorBoard"
 				(path "/c85d256f-82d8-4180-ad51-faa565e237b8/421006c7-5c19-4fe4-b045-335315607d2c"
-					(reference "J?")
+					(reference "J5")
 					(unit 1)
 				)
@@
 		(dnp no)
 		(fields_autoplaced yes)
-		(property "Reference" "#PWR039"
+		(property "Reference" "#PWR041"
 			(at 50.8 142.24 0)
 			(effects
@@
 			(project "PCB001-0A_processorBoard"
 				(path "/c85d256f-82d8-4180-ad51-faa565e237b8/421006c7-5c19-4fe4-b045-335315607d2c"
-					(reference "#PWR039")
+					(reference "#PWR041")
 					(unit 1)
 				)
@@
 		(dnp no)
 		(fields_autoplaced yes)
-		(property "Reference" "J?"
+		(property "Reference" "J4"
 			(at 43.18 107.95 0)
 			(effects
@@
 		(pin "3"
 		)
+		(instances
+			(project "PCB001-0A_processorBoard"
+				(path "/c85d256f-82d8-4180-ad51-faa565e237b8/421006c7-5c19-4fe4-b045-335315607d2c"
+					(reference "J4")
+					(unit 1)
+				)
+			)
+		)
 	)
 	(symbol
@@
 		(dnp no)
 		(fields_autoplaced yes)
-		(property "Reference" "#PWR042"
+		(property "Reference" "#PWR038"
 			(at 50.8 58.42 0)
 			(effects
@@
 		(pin "1"
 		)
+		(instances
+			(project "PCB001-0A_processorBoard"
+				(path "/c85d256f-82d8-4180-ad51-faa565e237b8/421006c7-5c19-4fe4-b045-335315607d2c"
+					(reference "#PWR038")
+					(unit 1)
+				)
+			)
+		)
 	)
 	(symbol
@@
 		(dnp no)
 		(fields_autoplaced yes)
-		(property "Reference" "#PWR040"
+		(property "Reference" "#PWR039"
 			(at 50.8 97.79 0)
 			(effects
@@
 			(project "PCB001-0A_processorBoard"
 				(path "/c85d256f-82d8-4180-ad51-faa565e237b8/421006c7-5c19-4fe4-b045-335315607d2c"
-					(reference "#PWR040")
+					(reference "#PWR039")
 					(unit 1)
 				)
@@
 		(on_board yes)
 		(dnp no)
-		(property "Reference" "R?"
+		(property "Reference" "R14"
 			(at 88.9 63.5 0)
 			(effects
@@
 			(project "PCB001-0A_processorBoard"
 				(path "/c85d256f-82d8-4180-ad51-faa565e237b8/421006c7-5c19-4fe4-b045-335315607d2c"
-					(reference "R?")
+					(reference "R14")
 					(unit 1)
 				)
@@
 		(on_board yes)
 		(dnp no)
-		(property "Reference" "U?"
+		(property "Reference" "U6"
 			(at 40.64 72.3899 0)
 			(effects
@@
 		(pin "8"
 		)
-	)
+		(instances
+			(project "PCB001-0A_processorBoard"
+				(path "/c85d256f-82d8-4180-ad51-faa565e237b8/421006c7-5c19-4fe4-b045-335315607d2c"
+					(reference "U6")
+					(unit 1)
+				)
+			)
+		)
+	)
