File: ECAD/Designs/PCB001_processorBoard/PCB001-0A_processorBoard/power_supply.kicad_sch (KiCad schematic)
At the start: 9 parts, among them J16 EXT_PWR, J17 PWR_SW, U7 LM66200, U8 AZ1117-3.3

Commit message: updated schematics
Parts:
- removed J16: EXT_PWR, Connector_JST:JST_PH_B2B-PH-K_1x02_P2.00mm_Vertical, symbol Connector_Generic:Conn_01x02
- removed U8: AZ1117-3.3, Package_TO_SOT_SMD:SOT-223, symbol Regulator_Linear:AZ1117-3.3
- added U9: TLV75533PDRV, Package_SON:WSON-6-1EP_2x2mm_P0.65mm_EP1x1.6mm, symbol Regulator_Linear:TLV75533PDRV
- renumbered C32 to C35, C33 to C36, C34 to C37, J17 to J16, R15 to R16, R16 to R17, U7 to U8
Connections:
- net +3V3: now also U9.1 (OUT)
- net +5V: now also C35.1, R17.1, U8.2 (VOUT), U8.7 (VOUT), U9.4 (EN), U9.6 (IN); no longer J16.2 (Pin_2), U8.3 (VIN1)
- net GND: now also U9.3 (GND), U9.7 (GND)
- new net 5V IN: J16.2 (Pin_2), U8.3 (VIN1)
